File: Schematics/AD2_extension/Experimental_Kit.kicad_sch (KiCad schematic)
At the start: 37 parts, among them J1 I2C, J10 AD2, J11 CN7, J12 CN10, J13 SPI_5V, J2 Keypad, J3 W2, J4 W1, J5 LCD, J6 SPI_3V3, J7 PWM, J8 PWM, J9 AREF, Q1 2N7002, Q2 2N7002, Q3 2N7002, Q4 2N7002, U1 TXU0304PW

Commit message: AD2_extension: 보호회로·I2C 버스·Feather 5V 추가, DRC/ERC 무시 항목 0
회로도
- W1/W2 입력 보호: 직렬 1k + BAT54S 클램프, AD2 V+ -> AREF 직렬 4.7k
- IOREF 점퍼를 쇼트키 D3(+3V3 -> IOREF)로 교체
- LCD 시프터와 AD2 I2C를 UNO SDA/SCL, Nucleo PB9/PB8, Feather SDA/SCL 공용 버스로 이전
- U1(TXU0304) OE -> IOREF, MISO 직렬 R13 2.2k
- Feather USB -> D4 -> +5V
- J10/J11/J12 심볼을 필터를 맞춘 프로젝트 사본으로 교체

PCB
- 점퍼 재배치(Nucleo 외곽 밖), W1/W2 정렬, 신규 부품 배치·배선
- 상면 GND 붓기와 스티칭 비아 추가, 배선 직선/45도 정리
- 실크 정리, J10 기판 가장자리용 풋프린트, MS1 코트야드 면제
- ERC/DRC 위반 0, 무시 항목 0

Co-Authored-By: Claude Opus 5.5 <noreply@anthropic.com>
Claude-Session: https://claude.ai/code/session_0124difPG7KsZZNpLXnsU8d2
Parts:
- added D4: 1N5819HW, Diode_SMD:D_SOD-123, symbol AD2_extension:D_Schottky
- J10: footprint Connector_PinSocket_2.54mm:PinSocket_2x15_P2.54mm_Horizontal -> AD2_extension:PinSocket_2x15_P2.54mm_Horizontal_BoardEdge; symbol Connector_Generic:Conn_02x15_Odd_Even -> AD2_extension:Conn_02x15_AD2
- J11, J12: symbol Connector_Generic:Conn_02x19_Odd_Even -> AD2_extension:Conn_02x19_Morpho
Connections:
- net +5V: now also D4.1 (K)
- net FEATHER_USB: now reaches MS1.26 (USB)
- net FEATHER_USB: now also D4.2 (A)
- no-connect marks 49 -> 48
Other:
- note removed: "U1 TXU0304: A1-A3 -> B1-B3 (SCK, MOSI, CS), B4 -> A4 (MISO). VCCA = IOREF, VCCB = +3V3"
- moved on the sheet: R13

Commit message: AD2_extension: 회로도 정리 및 PCB 동기화, README에 이동 경로 추가
- 회로도 정리 반영, PCB 업데이트(FEATHER_USB 넷 → Net-(D4-A))
- ERC 0, DRC 0, 미연결 0, 회로도-PCB 패리티 0
- README: Schematics/AD2_extension 항목 추가(01_Lectures 저장소에서 이동)

Co-Authored-By: Claude Opus 5.5 <noreply@anthropic.com>
Claude-Session: https://claude.ai/code/session_0124difPG7KsZZNpLXnsU8d2
Connections:
- net FEATHER_USB: no longer names the net of D4.2 (A), MS1.26 (USB)
Changed lines of the file:
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@@
 	(wire
 		(pts
+			(xy 177.8 109.22) (xy 180.34 109.22)
+		)
+		(stroke
+			(width 0)
+			(type default)
+		)
+	)
+	(wire
+		(pts
 			(xy 124.46 130.81) (xy 120.65 130.81)
 		)
@@
 	(wire
 		(pts
+			(xy 312.42 220.98) (xy 326.39 220.98)
+		)
+		(stroke
+			(width 0)
+			(type default)
+		)
+	)
+	(wire
+		(pts
 			(xy 351.79 215.9) (xy 364.49 215.9)
 		)
@@
 	(wire
 		(pts
+			(xy 180.34 120.65) (xy 165.1 120.65)
+		)
+		(stroke
+			(width 0)
+			(type default)
+		)
+	)
+	(wire
+		(pts
 			(xy 260.35 58.42) (xy 271.78 58.42)
 		)
@@
 	(wire
 		(pts
-			(xy 165.1 124.46) (xy 165.1 129.54)
-		)
-		(stroke
-			(width 0)
-			(type default)
-		)
-	)
-	(wire
-		(pts
 			(xy 185.42 124.46) (xy 185.42 129.54)
 		)
@@
 	(wire
 		(pts
-			(xy 312.42 220.98) (xy 326.39 220.98)
-		)
-		(stroke
-			(width 0)
-			(type default)
-		)
-	)
-	(wire
-		(pts
 			(xy 323.85 48.26) (xy 326.39 48.26)
 		)
@@
 	(wire
 		(pts
-			(xy 182.88 109.22) (xy 177.8 109.22)
-		)
-		(stroke
-			(width 0)
-			(type default)
-		)
-	)
-	(wire
-		(pts
 			(xy 36.83 110.49) (xy 46.99 110.49)
 		)
@@
 	(wire
 		(pts
+			(xy 180.34 109.22) (xy 180.34 120.65)
+		)
+		(stroke
+			(width 0)
+			(type default)
+		)
+	)
+	(wire
+		(pts
 			(xy 283.21 50.8) (xy 283.21 48.26)
 		)
@@
 	(wire
 		(pts
+			(xy 165.1 120.65) (xy 165.1 129.54)
+		)
+		(stroke
+			(width 0)
+			(type default)
+		)
+	)
+	(wire
+		(pts
 			(xy 172.72 142.24) (xy 172.72 147.32)
 		)
@@
 		)
 	)
-	(label "FEATHER_USB"
-		(at 35.56 64.77 0)
-		(effects
-			(font
-				(size 1.27 1.27)
-			)
-			(justify left bottom)
-		)
-	)
 	(label "LCD_SCL"
 		(at 339.09 139.7 180)
@@
 		)
 	)
-	(label "Vp"
-		(at 182.88 109.22 0)
-		(effects
-			(font
-				(size 1.27 1.27)
-			)
-			(justify left bottom)
-		)
-	)
 	(label "DIO5"
 		(at 304.8 73.66 180)
@@
 		)
 	)
+	(label "MISO_IO"
+		(at 321.31 220.98 180)
+		(effects
+			(font
+				(size 1.27 1.27)
+			)
+			(justify right bottom)
+		)
+	)
 	(label "DIO8"
 		(at 154.94 64.77 180)
@@
 		)
 	)
-	(label "MISO_IO"
-		(at 312.42 220.98 180)
-		(effects
-			(font
-				(size 1.27 1.27)
-			)
-			(justify right bottom)
-		)
-	)
